File: hw/poseidon.brd (EAGLE design)
At the start: 115.5 x 116.5 mm, 162 parts, among them IC1 MCP1703DB, J1 DCJ0202, Q1 IRF512, Q10 IRF512, Q11 IRF512, Q12 IRF512, Q13 IRF512, Q14 IRF512, Q15 IRF512, Q16 IRF512, Q17 IRF512, Q18 IRF512, Q19 IRF512, Q2 IRF512, Q3 IRF512, Q4 IRF512, Q5 IRF512, Q6 IRF512, Q7 IRF512, Q8 IRF512, Q9 IRF512, T1 2N5088, T10 2N5088, T11 2N5088, T12 2N5088, T13 2N5088, T14 2N5088, T15 2N5088, T16 2N5088, T2 2N5088, T3 2N5088, T4 2N5088, T5 2N5088, T6 2N5088, T7 2N5088, T8 2N5088, T9 2N5088, X1 B4B-ZR, X2 1296-T10, X3 22-23-2041, X4 22-23-2041, X5 22-23-2021

Commit message: Fixed problems with first revision, including barrel jack polarity
Also tidied up labels, connected extra vias to ground, created
test points for power rails. Still need to fix water level sensor
connector, which is currently too small.
Parts:
- removed THERM_D15: CREE-XT-E-WHITE, leds:CREE-XT-E
- added D19: LED0603, leds:LED-0603
- D15: value LED0603 -> CREE-XT-E-WHITE; device leds:LED-0603 -> leds:CREE-XT-E
- moved D15 61.0 mm to (16.5, 33.0), flipped to the bottom, turned to 0 degrees
Connections:
- net GND: now also J1.3; no longer J1.1
- net N$26: now also D19.A; no longer D15.A
- net N$5: now also D19.C; no longer D15.C
- net N$59: now also D15.K; no longer THERM_D15.K
- net THERM_D15: now also D15.THERMAL; no longer THERM_D15.THERMAL
- net VCC: now also D15.A, J1.1; no longer J1.3, THERM_D15.A
Routing:
- net GND: track 721.1 -> 732.5 mm, vias 15 -> 25
- net VCC: track 726.8 -> 733.4 mm, vias 8 -> 9
- net +3V3: vias 6 -> 7
Other:
- board text added: "3.3V"
- board text added: "5V"
- board text added: "GND"
- board text added: "Raspberry Pi Zero W"
- board text added: "STM32"
- board text added: "Test"
- board text added: "v0.2 - April 2019 - C. J. Blocker"
- board text removed: "v0.1 - Jan 2019 - C. J. Blocker"
